Commit message: add imu to sensors rename everything to test instead of xacro

File: reppy_bot_urdf/urdf/sensors.xacro (robot description, xacro)
@@ -5,15 +5,16 @@
        xmlns:xacro="http://ros.org/wiki/xacro"
 >
-<xacro:macro name="gps_receiver" params="id
-	 									 frame_id
-										 topic_name
-										 parent_link
-										 x y z
-										 velocity_topic_name
-										 reference_latitude
-										 reference_longitude
-										 reference_heading
-										 reference_altitude
-										">
+<xacro:macro name="gps_receiver"
+params= "id
+		 frame_id
+		 topic_name
+		 parent_link
+		 x y z
+		 velocity_topic_name
+		 reference_latitude
+		 reference_longitude
+		 reference_heading
+		 reference_altitude
+		">
 	<link name="gps_receiver_link${id}">
 		<visual>
@@ -25,19 +26,4 @@
 			</material>
 		</visual>
-		<collision>
-			<geometry>
-				<box size="0.04 0.04 0.04" />
-			</geometry>
-		</collision>
-		<inertial>
-	            <mass value="1.0"/>
-	            <origin xyz="0.0 0.0 0.0"/>
-	            <inertia ixx="0.1"
-	                     iyy="0.1"
-	                     izz="0.1"
-	  	            	 iyz="0.0"
-			             ixy="0.0"
-			             ixz="0.0"/>
-	    </inertial>
 	</link>
 	<joint name="gps_receiver_joint${id}" type="fixed">
@@ -60,26 +46,34 @@
 </gazebo>
 </xacro:macro>
-	<xacro:macro name="test_sensors">
-	  <gazebo>
-	  <!-- IMU -->
+<xacro:macro name="imu" params="id
+								topic_name
+								parent_link
+								x y z roll pitch yaw
+								gaussian_noise
+								">
+<link name="imu_link${id}">
+	<visual>
+		<geometry>
+			<box size="0.02 0.02 0.02" />
+		</geometry>
+		<material name="Yellow">
+			<color rgba="1 1 0 1"/>
+		</material>
+	</visual>
+</link>
+<joint name="imu_joint${id}" type="fixed">
+	<parent link="${parent_link}" />
+	<child link="imu_link${id}" />
+	<origin xyz="${x} ${y} ${z}" rpy="${roll} ${pitch} ${yaw}" />
+</joint>
+<gazebo>
 	  <plugin name="imu_controller" filename="libgazebo_ros_imu.so">
-			<bodyName>base_link</bodyName>
-			<topicName>imu</topicName>
-			<gaussianNoise>2.89e-08</gaussianNoise>
-			<xyzOffsets>-0.086632 0 0.12</xyzOffsets>
+			<bodyName>imu_link${id}</bodyName>
+			<topicName>${topic_name}</topicName>
+			<gaussianNoise>${gaussian_noise}</gaussianNoise>
+			<xyzOffsets>0 0 0</xyzOffsets>
 			<rpyOffsets>0 0 0</rpyOffsets>
 	  </plugin>
-	  <!-- GPS -->
-	  <plugin name="gps_controller" filename="libhector_gazebo_ros_gps.so">
-	  	<bodyName>base_link</bodyName>
-	  	<frameId>world</frameId>
-	  	<topicName>fix</topicName>
-	  	<velocityTopicName>fix_velocity</velocityTopicName>
-	  	<referenceLatitude>49.9</referenceLatitude>
-	  	<referenceLongitude>8.9</referenceLongitude>
-	  	<referenceHeading>0</referenceHeading>
-	  	<referenceAltitude>0</referenceAltitude>
-	  </plugin>
-	  </gazebo>
-	</xacro:macro>
+</gazebo>
+</xacro:macro>
 </robot>

File: reppy_bot_urdf/urdf/test_bot.xacro (robot description, xacro)
@@ -113,9 +113,20 @@
 					 x="0" y="0" z="0"
 					 frame_id="world"
-					 topic_name="fix"
-					 velocity_topic_name="fix_vel"
+					 topic_name="/fix"
+					 velocity_topic_name="/fix_vel"
 					 reference_latitude="49"
 					 reference_longitude="8"
 					 reference_heading="0"
 					 reference_altitude="0"/>
+<xacro:imu 	id="0"
+			topic_name="/imu"
+			parent_link="chassis"
+			x="${wheel_base_center_x}"
+			y="0"
+			z="0"
+			roll="0"
+			pitch="0"
+			yaw="0"
+			gaussian_noise="2.89e-08"
+			/>
 </robot>
