Commit message: add gps, camera, imu, rplidar

File: reppy_bot_urdf/urdf/gps.xacro (robot description, xacro)
@@ -5,4 +5,7 @@
        xmlns:xacro="http://ros.org/wiki/xacro"
 >
+<!--
+	GPS
+-->
 <xacro:macro name="gps_receiver"
 params= "id
@@ -46,34 +49,3 @@
 </gazebo>
 </xacro:macro>
-<xacro:macro name="imu" params="id
-								topic_name
-								parent_link
-								x y z roll pitch yaw
-								gaussian_noise
-								">
-<link name="imu_link${id}">
-	<visual>
-		<geometry>
-			<box size="0.02 0.02 0.02" />
-		</geometry>
-		<material name="Yellow">
-			<color rgba="1 1 0 1"/>
-		</material>
-	</visual>
-</link>
-<joint name="imu_joint${id}" type="fixed">
-	<parent link="${parent_link}" />
-	<child link="imu_link${id}" />
-	<origin xyz="${x} ${y} ${z}" rpy="${roll} ${pitch} ${yaw}" />
-</joint>
-<gazebo>
-	  <plugin name="imu_controller" filename="libgazebo_ros_imu.so">
-			<bodyName>imu_link${id}</bodyName>
-			<topicName>${topic_name}</topicName>
-			<gaussianNoise>${gaussian_noise}</gaussianNoise>
-			<xyzOffsets>0 0 0</xyzOffsets>
-			<rpyOffsets>0 0 0</rpyOffsets>
-	  </plugin>
-</gazebo>
-</xacro:macro>
 </robot>

File: reppy_bot_urdf/urdf/test_bot.xacro (robot description, xacro)
@@ -6,6 +6,9 @@
 <xacro:include filename="$(find reppy_bot_urdf)/urdf/consts.xacro"/>
 <xacro:include filename="$(find reppy_bot_urdf)/urdf/diff_drive_setup.xacro"/>
-<xacro:include filename="$(find reppy_bot_urdf)/urdf/sensors.xacro"/>
-<!-- Simple Robot Settings -->
+<xacro:include filename="$(find reppy_bot_urdf)/urdf/gps.xacro"/>
+<xacro:include filename="$(find reppy_bot_urdf)/urdf/imu.xacro"/>
+<xacro:include filename="$(find reppy_bot_urdf)/urdf/rplidar.xacro"/>
+<xacro:include filename="$(find reppy_bot_urdf)/urdf/camera.xacro"/>
+	<!-- Simple Robot Settings -->
 <xacro:property name="chassis_height" value="0.15"/>
 <xacro:property name="chassis_width"  value="${chassis_height*1.618}"/>
@@ -130,3 +133,36 @@
 			gaussian_noise="2.89e-08"
 			/>
+<xacro:rplidar id="0"
+		topic_name="/laser/scan"
+		frame_name="laser"
+		parent_link="chassis"
+		x="0" y="0" z="${chassis_height/2}" roll="0" pitch="0" yaw="0"
+		update_rate="5.5"
+		visualize="false"
+/>
+<xacro:cam
+		id="0"
+		parent_link="chassis"
+		x="${chassis_len}" y="0" z="0" roll="0" pitch="-0.01" yaw="${const_pi}"
+		always_on="true"
+		topic_video_name="camera0"
+		topic_camera_info="camera0_info"
+		frame_name="camera0"
+		image_width="640"
+		image_height="480"
+		image_format="R8G8B8"
+		clip_near="0.02"
+		clip_far="300"
+		noise_type="gausian"
+		noise_mean="0.0"
+		noise_std_dev="0.007"
+		fov="0.873"
+		hack_baseline="0.07"
+		dist_K1="0.0"
+		dist_K2="0.0"
+		dist_K3="0.0"
+		dist_T1="0.0"
+		dist_T2="0.0"
+		update_rate="30"
+        />
 </robot>
