Commit message: fix camera

File: reppy_bot_urdf/urdf/camera.xacro (robot description, xacro)
@@ -10,6 +10,4 @@
 								x y z roll pitch yaw
 								always_on
-								topic_video_name
-								topic_camera_info
 								frame_name
 								image_width
@@ -37,5 +35,5 @@
 			<box size="0.02 0.02 0.02" />
 		</geometry>
-		<material name="Gazebo/FlatBlack">
+		<material name="Black">
 			<color rgba="0.0 0.0 0.0 1.0"/>
 		</material>
@@ -55,4 +53,5 @@
 </joint>
 <gazebo reference="camera${id}_link">
+	<material value="Gazebo/FlatBlack" />
 	<sensor type="camera" name="camera${id}">
 		<update_rate>${update_rate}</update_rate>
@@ -78,6 +77,6 @@
 			<updateRate>${update_rate}</updateRate>
 			<cameraName>camera${id}</cameraName>
-			<imageTopicName>${topic_video_name}</imageTopicName>
-			<cameraInfoTopicName>${topic_camera_info}</cameraInfoTopicName>
+			<imageTopicName>image_raw</imageTopicName>
+			<cameraInfoTopicName>camera_info</cameraInfoTopicName>
 			<frameName>${frame_name}</frameName>
 			<hackBaseline>${hack_baseline}</hackBaseline>
@@ -89,5 +88,5 @@
 		</plugin>
 	</sensor>
-</gazebo><!---->
+</gazebo>
 </xacro:macro>
 </robot>

File: reppy_bot_urdf/urdf/test_bot.xacro (robot description, xacro)
@@ -4,20 +4,20 @@
        xmlns:interface="http://playerstage.sourceforge.net/gazebo/xmlschema/#interface"
        xmlns:xacro="http://ros.org/wiki/xacro" name="reppy_bot">
-<xacro:include filename="$(find reppy_bot_urdf)/urdf/consts.xacro"/>
+<xacro:include filename="$(find reppy_bot_urdf)/urdf/consts.xacro"			/>
 <xacro:include filename="$(find reppy_bot_urdf)/urdf/diff_drive_setup.xacro"/>
-<xacro:include filename="$(find reppy_bot_urdf)/urdf/gps.xacro"/>
-<xacro:include filename="$(find reppy_bot_urdf)/urdf/imu.xacro"/>
-<xacro:include filename="$(find reppy_bot_urdf)/urdf/rplidar.xacro"/>
-<xacro:include filename="$(find reppy_bot_urdf)/urdf/camera.xacro"/>
-	<!-- Simple Robot Settings -->
-<xacro:property name="chassis_height" value="0.15"/>
-<xacro:property name="chassis_width"  value="${chassis_height*1.618}"/>
-<xacro:property name="chassis_len"    value="${chassis_width+chassis_height}"/>
-<xacro:property name="chassis_floor_clearance" value="${chassis_height/(1.618*2)}"/>
-<xacro:property name="wheel_diameter" value="${chassis_len/(1.618*1.618)}"/>
-<xacro:property name="wheel_width" value="${chassis_width/(16.18)}"/>
-<xacro:property name="wheel_base_center_x" value="${chassis_len/(-1.618*3)}"/>
-<xacro:property name="caster_collision_x" value="${chassis_len/(1.618*2)}"/>
-<link name="base_link"/>
+<xacro:include filename="$(find reppy_bot_urdf)/urdf/gps.xacro"				/>
+<xacro:include filename="$(find reppy_bot_urdf)/urdf/imu.xacro"				/>
+<xacro:include filename="$(find reppy_bot_urdf)/urdf/rplidar.xacro"			/>
+<xacro:include filename="$(find reppy_bot_urdf)/urdf/camera.xacro"			/>
+<!-- Simple Robot Settings -->
+<xacro:property name="chassis_height"          value="0.15"                            />
+<xacro:property name="chassis_width"           value="${chassis_height*1.618}"         />
+<xacro:property name="chassis_len"             value="${chassis_width+chassis_height}" />
+<xacro:property name="chassis_floor_clearance" value="${chassis_height/(1.618*2)}"     />
+<xacro:property name="wheel_diameter"          value="${chassis_len/(1.618*1.618)}"    />
+<xacro:property name="wheel_width"             value="${chassis_width/(16.18)}"        />
+<xacro:property name="wheel_base_center_x"     value="${chassis_len/(-1.618*3)}"       />
+<xacro:property name="caster_collision_x"      value="${chassis_len/(1.618*2)}"        />
+<link name="base_link" />
 <link name="chassis">
 	<visual>
@@ -112,57 +112,66 @@
 	 ros_plugin_publish_wheel_tf="true"
 	 ros_plugin_publish_tf="1" />
-<xacro:gps_receiver  id="0"
-					 parent_link="chassis"
-					 x="0" y="0" z="0"
-					 frame_id="world"
-					 topic_name="/fix"
-					 velocity_topic_name="/fix_vel"
-					 reference_latitude="49"
-					 reference_longitude="8"
-					 reference_heading="0"
-					 reference_altitude="0"/>
-<xacro:imu 	id="0"
-			topic_name="/imu"
-			parent_link="chassis"
-			x="${wheel_base_center_x}"
-			y="0"
-			z="0"
-			roll="0"
-			pitch="0"
-			yaw="0"
-			gaussian_noise="2.89e-08"
-			/>
+<xacro:gps_receiver
+		id="0"
+		parent_link="chassis"
+		x="0" y="0" z="0"
+		frame_id="world"
+		topic_name="/fix"
+		velocity_topic_name="/fix_vel"
+		reference_latitude="49"
+		reference_longitude="8"
+		reference_heading="0"
+		reference_altitude="0"/>
+<xacro:imu
+		id="0"
+		topic_name="/imu"
+		parent_link="chassis"
+		x="${wheel_base_center_x}"
+		y="0"
+		z="0"
+		roll="0"
+		pitch="0"
+		yaw="0"
+		gaussian_noise="2.89e-08"
+		/>
 <xacro:rplidar id="0"
 		topic_name="/laser/scan"
 		frame_name="laser"
 		parent_link="chassis"
-		x="0" y="0" z="${chassis_height/2}" roll="0" pitch="0" yaw="0"
+		x="0"
+        y="0"
+        z="${chassis_height/2}"
+	    roll="0"
+	    pitch="0"
+        yaw="0"
 		update_rate="5.5"
-		visualize="false"
-/>
+		visualize="false" />
 <xacro:cam
-		id="0"
-		parent_link="chassis"
-		x="${chassis_len}" y="0" z="0" roll="0" pitch="-0.01" yaw="${const_pi}"
-		always_on="true"
-		topic_video_name="camera0"
-		topic_camera_info="camera0_info"
-		frame_name="camera0"
-		image_width="640"
-		image_height="480"
-		image_format="R8G8B8"
-		clip_near="0.02"
-		clip_far="300"
-		noise_type="gausian"
-		noise_mean="0.0"
-		noise_std_dev="0.007"
-		fov="0.873"
-		hack_baseline="0.07"
-		dist_K1="0.0"
-		dist_K2="0.0"
-		dist_K3="0.0"
-		dist_T1="0.0"
-		dist_T2="0.0"
-		update_rate="30"
+		id               ="0"
+		parent_link      ="chassis"
+		x                ="${chassis_len/2}"
+	    y                ="0"
+        z                ="0"
+        roll             ="0"
+        pitch            ="-0.01"
+        yaw              ="0"
+		always_on        ="true"
+		frame_name       ="camera0"
+		image_width      ="640"
+		image_height     ="480"
+		image_format     ="R8G8B8"
+		clip_near        ="0.02"
+		clip_far         ="300"
+		noise_type       ="gausian"
+		noise_mean       ="0.0"
+		noise_std_dev    ="0.007"
+		fov              ="0.873"
+		hack_baseline    ="0.07"
+		dist_K1          ="0.0"
+		dist_K2          ="0.0"
+		dist_K3          ="0.0"
+		dist_T1          ="0.0"
+		dist_T2          ="0.0"
+		update_rate      ="30"
         />
 </robot>

Commit message: add robot namespace support

File: reppy_bot_urdf/urdf/camera.xacro (robot description, xacro)
@@ -7,4 +7,5 @@
 <xacro:macro name="cam" params="
 	 							id
+	 							robot_namespace
 								parent_link
 								x y z roll pitch yaw
@@ -74,4 +75,5 @@
 		</camera>
 		<plugin name="camera_sensor" filename="libgazebo_ros_camera.so">
+			<robotNamespace>${robot_namespace}</robotNamespace>
 			<alwaysOn>${always_on}</alwaysOn>
 			<updateRate>${update_rate}</updateRate>

File: reppy_bot_urdf/urdf/diff_drive_setup.xacro (robot description, xacro)
@@ -68,4 +68,5 @@
 		<plugin name="${ros_plugin_controller_name}" filename="libgazebo_ros_diff_drive.so">
 			<robotBaseFrame>${base_frame}</robotBaseFrame>
+			<robotNamespace>${robot_namespace}</robotNamespace>
 			<wheelSeparation>${wheel_separation}</wheelSeparation>
 			<wheelDiameter>${wheel_diameter}</wheelDiameter>

File: reppy_bot_urdf/urdf/gps.xacro (robot description, xacro)
@@ -10,4 +10,5 @@
 <xacro:macro name="gps_receiver"
 params= "id
+		 robot_namespace
 		 frame_id
 		 topic_name
@@ -20,5 +21,5 @@
 		 reference_altitude
 		">
-	<link name="gps_receiver_link${id}">
+	<link name="gps${id}_receiver_link">
 		<visual>
 			<geometry>
@@ -30,13 +31,14 @@
 		</visual>
 	</link>
-	<joint name="gps_receiver_joint${id}" type="fixed">
+	<joint name="gps${id}_receiver_joint" type="fixed">
 		<parent link="${parent_link}" />
-		<child link="gps_receiver_link${id}" />
+		<child link="gps${id}_receiver_link" />
 		<origin xyz="${x} ${y} ${z}" rpy="0 0 0" />
 	</joint>
 <gazebo>
-	<plugin name="gps_controller${id}"
+	<plugin name="gps${id}_controller"
 		    filename="libhector_gazebo_ros_gps.so">
-		<bodyName>gps_receiver_link${id}</bodyName>
+		<robotNamespace>${robot_namespace}</robotNamespace>
+		<bodyName>gps${id}_receiver_link</bodyName>
 		<frameId>${frame_id}</frameId>
 		<topicName>${topic_name}</topicName>

File: reppy_bot_urdf/urdf/imu.xacro (robot description, xacro)
@@ -9,4 +9,5 @@
 -->
 <xacro:macro name="imu" params="id
+								robot_namespace
 								topic_name
 								parent_link
@@ -14,5 +15,5 @@
 								gaussian_noise
 								">
-<link name="imu_link${id}">
+<link name="imu${id}_link">
 	<visual>
 		<geometry>
@@ -24,12 +25,13 @@
 	</visual>
 </link>
-<joint name="imu_joint${id}" type="fixed">
+<joint name="imu${id}_joint" type="fixed">
 	<parent link="${parent_link}" />
-	<child link="imu_link${id}" />
+	<child link="imu${id}_link" />
 	<origin xyz="${x} ${y} ${z}" rpy="${roll} ${pitch} ${yaw}" />
 </joint>
 <gazebo>
 	  <plugin name="imu_controller" filename="libgazebo_ros_imu.so">
-			<bodyName>imu_link${id}</bodyName>
+			<robotNamespace>${robot_namespace}</robotNamespace>
+			<bodyName>imu${id}_link</bodyName>
 			<topicName>${topic_name}</topicName>
 			<gaussianNoise>${gaussian_noise}</gaussianNoise>

File: reppy_bot_urdf/urdf/rplidar.xacro (robot description, xacro)
@@ -7,4 +7,5 @@
 <xacro:include filename="$(find reppy_bot_urdf)/urdf/consts.xacro"/>
 <xacro:macro name="rplidar" params="id
+								robot_namespace
 								topic_name
 								frame_name
@@ -70,5 +71,6 @@
       </ray>
       <plugin name="gazebo_ros_head_rplidar${id}_controller" filename="libgazebo_ros_gpu_laser.so">
-        <topicName>${topic_name}</topicName>
+        <robotNamespace>${robot_namespace}</robotNamespace>
+      	<topicName>${topic_name}</topicName>
         <frameName>rplidar${id}_link</frameName>
       </plugin>

File: reppy_bot_urdf/urdf/test_bot.xacro (robot description, xacro)
@@ -19,4 +19,5 @@
 <xacro:property name="wheel_base_center_x"     value="${chassis_len/(-1.618*3)}"       />
 <xacro:property name="caster_collision_x"      value="${chassis_len/(1.618*2)}"        />
+<xacro:property name="robot_namespace" value="/" />
 <link name="base_link" />
 <link name="chassis">
@@ -88,5 +89,5 @@
 <xacro:diff_drive_setup
 	 base_frame="base_link"
-	 robot_namespace=""
+	 robot_namespace="${robot_namespace}"
 	 wheel_base_center_x="${wheel_base_center_x}"
      wheel_separation ="${chassis_width}"
@@ -114,4 +115,5 @@
 <xacro:gps_receiver
 		id="0"
+	 	robot_namespace="${robot_namespace}"
 		parent_link="chassis"
 		x="0" y="0" z="0"
@@ -125,4 +127,5 @@
 <xacro:imu
 		id="0"
+	 	robot_namespace=""
 		topic_name="/imu"
 		parent_link="chassis"
@@ -136,4 +139,5 @@
 		/>
 <xacro:rplidar id="0"
+	 	robot_namespace="${robot_namespace}"
 		topic_name="/laser/scan"
 		frame_name="laser"
@@ -149,4 +153,5 @@
 <xacro:cam
 		id               ="0"
+	 	robot_namespace  ="${robot_namespace}"
 		parent_link      ="chassis"
 		x                ="${chassis_len/2}"
