Commit message: xacro files for robot still buggy not working in gazebo

File: reppy_bot_urdf/urdf/diff_drive_setup.xacro (robot description, xacro)
@@ -4,7 +4,9 @@
        xmlns:interface="http://playerstage.sourceforge.net/gazebo/xmlschema/#interface"
        xmlns:xacro="http://ros.org/wiki/xacro">
-<xacro:include filename="$(find reppy_bot_urdf)/defs/consts.xacro"/>
+<xacro:include filename="$(find reppy_bot_urdf)/urdf/consts.xacro"/>
+<xacro:include filename="$(find reppy_bot_urdf)/urdf/diff_drive_wheel.xacro"/>
 <xacro:macro name="diff_drive_setup"
 	         params="base_frame
+					 robot_namespace
 	                 wheel_base_center_x
 	                 wheel_separation
@@ -12,4 +14,12 @@
 	                 wheel_torque
 					 wheel_acceleration
+					 wheel_joint_limit_vel
+					 wheel_joint_limit_effort
+					 wheel_friction1
+	                 wheel_friction2
+	  				 wheel_contact_damping
+	                 wheel_contact_stiffness
+	 				 wheel_mass
+					 wheel_width
 	                 cmd_topic
 					 odom_topic
@@ -23,4 +33,36 @@
 					 ros_plugin_publish_tf
 	                 ">
+		<xacro:diff_drive_wheel
+			                 name="${ros_plugin_controller_name}_wheel_left"
+						     base_frame="${base_frame}"
+			                 radius="${wheel_diameter/2}"
+			                 width="${wheel_width}"
+							 mass="${wheel_mass}"
+							 origin_x="${wheel_base_center_x}"
+							 origin_y="${wheel_separation/2}"
+							 origin_z="${wheel_diameter/2}"
+							 limit_vel="${wheel_joint_limit_vel}"
+							 limit_effort="${wheel_joint_limit_effort}"
+							 contact_stiffness="${wheel_contact_stiffness}"
+							 contact_damping="${wheel_contact_damping}"
+		                     friction1="${wheel_friction1}"
+							 friction2="${wheel_friction2}"
+							 />
+		<xacro:diff_drive_wheel
+                 name="${ros_plugin_controller_name}_wheel_right"
+			     base_frame="${base_frame}"
+                 radius="${wheel_diameter/2}"
+                 width="${wheel_width}"
+				 mass="${wheel_mass}"
+				 origin_x="${wheel_base_center_x}"
+				 origin_y="-${wheel_separation/2}"
+				 origin_z="${wheel_diameter/2}"
+				 limit_vel="${wheel_joint_limit_vel}"
+				 limit_effort="${wheel_joint_limit_effort}"
+				 contact_stiffness="${wheel_contact_stiffness}"
+				 contact_damping="${wheel_contact_damping}"
+                 friction1="${wheel_friction1}"
+				 friction2="${wheel_friction2}"
+				 />
 	<gazebo>
 		<plugin name="${ros_plugin_controller_name}" filename="libgazebo_ros_diff_drive.so">
@@ -36,6 +78,6 @@
 			<updateRate>${ros_plugin_update_rate}</updateRate>
 			<odometrySource>${ros_plugin_odom_source}</odometrySource>
-			<leftJoint>${ros_plugin_controller_name}_left_wheel_joint</leftJoint>
-			<rightJoint>${ros_plugin_controller_name}_right_wheel_joint</rightJoint>
+			<leftJoint>${ros_plugin_controller_name}_wheel_left_joint</leftJoint>
+			<rightJoint>${ros_plugin_controller_name}_wheel_right_joint</rightJoint>
 			<rosDebugLevel>${debugLevel}</rosDebugLevel>
 			<publishWheelTF>${ros_plugin_publish_wheel_tf}</publishWheelTF>

File: reppy_bot_urdf/urdf/diff_drive_wheel.xacro (robot description, xacro)
@@ -4,10 +4,10 @@
        xmlns:interface="http://playerstage.sourceforge.net/gazebo/xmlschema/#interface"
        xmlns:xacro="http://ros.org/wiki/xacro">
-	<xacro:include filename="$(find reppy_bot_urdf)/defs/consts.xacro"/>
+	<xacro:include filename="$(find reppy_bot_urdf)/urdf/consts.xacro"/>
 	<xacro:macro name="diff_drive_wheel"
 			         params="name
-						     base_link
+						     base_frame
 			                 radius
-			                 thickness
+			                 width
 							 mass
 							 origin_x origin_y origin_z
@@ -22,6 +22,6 @@
 			<mass value="${mass}"/>
 			<origin xyz="0 0 0" rpy="${const_pi/2} 0 0" />
-		    <inertia  ixx="${1/4*mass*radius*radius+1/12*mass+thickness*thickness}"
-                      iyy="${1/4*mass*radius*radius+1/12*mass+thickness*thickness}"
+		    <inertia  ixx="${1/4*mass*radius*radius+1/12*mass+width*width}"
+                      iyy="${1/4*mass*radius*radius+1/12*mass+width*width}"
                       izz="${1/2*mass*radius*radius}"
 		    		  ixy = "0" ixz = "0" iyz = "0"  />
@@ -31,5 +31,5 @@
 			        rpy="${const_pi/2} 0 0"/>
 			<geometry>
-				<cylinder radius="${radius}" length="${thickness}"/>
+				<cylinder radius="${radius}" length="${width}"/>
 			</geometry>
 			<material name="WheelBlack">
@@ -41,13 +41,13 @@
 			        rpy="${const_pi/2} 0 0"/>
 			<geometry>
-				<cylinder radius="${radius}" length="${thickness}"/>
+				<cylinder radius="${radius}" length="${width}"/>
 			</geometry>
 		</collision>
 		</link>
-		<joint name="${name}_joint" type="continuous">
+    <joint name="${name}_joint" type="continuous">
 		<axis xyz="0 1 0" />
 		<origin xyz="${origin_x} ${origin_y} ${origin_z}" py="0 0 0"/>
-    	<limit effort="${}" velocity="${limit_vel}" />
-   		<parent link="${base_link}"/>
+    	<limit effort="${limit_effort}" velocity="${limit_vel}" />
+   		<parent link="${base_frame}"/>
 		<child link="${name}"/>
 	</joint>

File: reppy_bot_urdf/urdf/reppy_bot.xacro (robot description, xacro)
@@ -3,15 +3,80 @@
        xmlns:controller="http://playerstage.sourceforge.net/gazebo/xmlschema/#controller"
        xmlns:interface="http://playerstage.sourceforge.net/gazebo/xmlschema/#interface"
-       xmlns:xacro="http://ros.org/wiki/xacro">
-<xacro:include filename="$(find reppy_bot_urdf)/defs/consts.xacro"/>
-<xacro:include filename="$(find reppy_bot_urdf)/defs/diff_drive_setup.xacro"/>
+       xmlns:xacro="http://ros.org/wiki/xacro" name="reppy_bot">
+<xacro:include filename="$(find reppy_bot_urdf)/urdf/consts.xacro"/>
+<xacro:include filename="$(find reppy_bot_urdf)/urdf/diff_drive_setup.xacro"/>
+<!-- Simple Robot Settings -->
+	<xacro:property name="wheel_diameter" value="0.05"/>
+	<xacro:property name="wheel_width" value="0.01"/>
+	<xacro:property name="wheel_base_center_x" value="-0.02"/>
+	<xacro:property name="wheel_separation" value="0.10"/>
+	<xacro:property name="chassis_width"  value="0.07"/>
+	<xacro:property name="chassis_len"    value="0.09"/>
+	<xacro:property name="chassis_height" value="0.04"/>
+    <xacro:property name="chassis_floor_clearance" value="0.02"/>
+    <xacro:property name="caster_collision_x" value="0.02"/>
+<link name="base_link"/>
+<link name="chassis">
+	<visual>
+		<geometry>
+			<box size="${chassis_len} ${chassis_width} ${chassis_height}" />
+		</geometry>
+	</visual>
+	<collision>
+		<geometry>
+			<box size="${chassis_len} ${chassis_width} ${chassis_height}" />
+		</geometry>
+	</collision>
+	<material>
+		<color rgba="0.0 0.0 1.0 1.0"/>
+	</material>
+</link>
+<gazebo reference="chassis">
+	<material name="Gazebo/Blue"/>
+</gazebo>
+<joint name="base_chassis_joint" type="fixed">
+	<parent link="base_link" />
+	<child link="chassis" />
+	<origin xyz="0 0 ${chassis_floor_clearance+chassis_height/2}" rpy="0 0 0" />
+</joint>
+<link name="caster_collision">
+	<visual>
+		<geometry>
+			<sphere radius="${chassis_floor_clearance}" />
+		</geometry>
+	</visual>
+	<collision>
+		<geometry>
+			<sphere radius="${chassis_floor_clearance}" />
+		</geometry>
+	</collision>
+	<material>
+		<color rgba="0.0 0.0 1.0 1.0"/>
+	</material>
+</link>
+<gazebo reference="caster_collision">
+	<material name="Gazebo/FlatBlack"/>
+</gazebo>
+<joint name="base_caster_col_joint" type="fixed">
+	<parent link="base_link" />
+	<child link="caster_collision" />
+	<origin xyz="${caster_collision_x} 0 ${chassis_floor_clearance}" rpy="0 0 0" />
+</joint>
 <xacro:diff_drive_setup
 	 base_frame="base_link"
 	 robot_namespace=""
-	 wheel_base_center_x="0"
-     wheel_separation ="0.070"
-     wheel_diameter="0.004"
+	 wheel_base_center_x="-0.02"
+     wheel_separation ="${chassis_width}"
+     wheel_diameter="${wheel_diameter}"
+	 wheel_width="${wheel_width}"
      wheel_torque="5"
 	 wheel_acceleration="1"
+	 wheel_joint_limit_vel="2"
+	 wheel_joint_limit_effort="2"
+	 wheel_friction1="100000"
+     wheel_friction2="1000"
+	 wheel_contact_damping="10"
+     wheel_contact_stiffness="10"
+	 wheel_mass="3"
      cmd_topic="/cmd_vel"
 	 odom_topic="odom"

Commit message: fix diff drive macro fix caster generation

File: reppy_bot_urdf/urdf/diff_drive_setup.xacro (robot description, xacro)
@@ -22,4 +22,5 @@
 	 				 wheel_mass
 					 wheel_width
+					 z_dist
 	                 cmd_topic
 					 odom_topic
@@ -41,5 +42,5 @@
 							 origin_x="${wheel_base_center_x}"
 							 origin_y="${(wheel_separation+wheel_width)/2}"
-							 origin_z="${wheel_diameter/2}"
+							 origin_z="${z_dist}"
 							 limit_vel="${wheel_joint_limit_vel}"
 							 limit_effort="${wheel_joint_limit_effort}"
@@ -57,5 +58,5 @@
 				 origin_x="${wheel_base_center_x}"
 				 origin_y="-${(wheel_separation+wheel_width)/2}"
-				 origin_z="${wheel_diameter/2}"
+				 origin_z="${z_dist}"
 				 limit_vel="${wheel_joint_limit_vel}"
 				 limit_effort="${wheel_joint_limit_effort}"

File: reppy_bot_urdf/urdf/test_bot.xacro (robot description, xacro)
@@ -59,5 +59,5 @@
 	<material value="Gazebo/FlatBlack" />
 </gazebo>
-<!--CASTER
+<!--CASTER -->
 <link name="caster_collision">
 	<visual>
@@ -85,42 +85,12 @@
     </inertial>
 </link>
--->
-<!--
 <gazebo reference="caster_collision">
 	<material value="Gazebo/FlatBlack"/>
 </gazebo>
 <joint name="base_caster_col_joint" type="fixed">
-	<parent link="base_link" />
+	<parent link="chassis" />
 	<child link="caster_collision" />
-	<origin xyz="${caster_collision_x} 0 ${chassis_floor_clearance}" rpy="0 0 0" />
+	<origin xyz="${caster_collision_x} 0 ${-(chassis_height/2)}" rpy="0 0 0" />
 </joint>
-<xacro:diff_drive_setup
-	 base_frame="base_link"
-	 robot_namespace="${robot_namespace}"
-	 wheel_base_center_x="${wheel_base_center_x}"
-     wheel_separation ="${chassis_width}"
-     wheel_diameter="${wheel_diameter}"
-	 wheel_width="${wheel_width}"
-     wheel_torque="5"
-	 wheel_acceleration="1"
-	 wheel_joint_limit_vel="2"
-	 wheel_joint_limit_effort="2"
-	 wheel_friction1="100000"
-     wheel_friction2="1000"
-	 wheel_contact_damping="100.0"
-     wheel_contact_stiffness="1000000.0"
-	 wheel_mass="3"
-     cmd_topic="/cmd_vel"
-	 odom_topic="odom"
-     odom_frame="odom"
-	 ros_plugin_always_on="true"
-	 ros_plugin_controller_name="diff_drv0"
-     ros_plugin_update_rate="100"
-	 ros_plugin_odom_source="encoder"
-	 ros_plugin_publish_wheel_joint_state="true"
-	 ros_plugin_publish_wheel_tf="true"
-	 ros_plugin_publish_tf="1" />
-	-->
-	 	<!--
 <xacro:gps_receiver
 		id="0"
@@ -196,4 +166,35 @@
 		update_rate      ="30"
         />
+<!--
+ DRIVE
+-->
+<xacro:diff_drive_setup
+	 base_frame="chassis"
+	 robot_namespace="${robot_namespace}"
+	 wheel_base_center_x="${wheel_base_center_x}"
+     wheel_separation ="${chassis_width}"
+     wheel_diameter="${wheel_diameter}"
+	 wheel_width="${wheel_width}"
+     wheel_torque="5"
+	 wheel_acceleration="1"
+	 wheel_joint_limit_vel="2"
+	 wheel_joint_limit_effort="2"
+	 wheel_friction1="100000"
+     wheel_friction2="1000"
+	 wheel_contact_damping="100.0"
+     wheel_contact_stiffness="1000000.0"
+	 wheel_mass="3"
+	 z_dist="${-((chassis_floor_clearance+chassis_height/2)-(wheel_diameter/2))}"
+     cmd_topic="/cmd_vel"
+	 odom_topic="odom"
+     odom_frame="odom"
+	 ros_plugin_always_on="true"
+	 ros_plugin_controller_name="diff_drv0"
+     ros_plugin_update_rate="100"
+	 ros_plugin_odom_source="encoder"
+	 ros_plugin_publish_wheel_joint_state="true"
+	 ros_plugin_publish_wheel_tf="true"
+	 ros_plugin_publish_tf="1" />
+	 	<!--
         	-->
 </robot>
