Commit message: rename reppy_bot to test_bot

File: reppy_bot_urdf/urdf/test_bot.xacro (robot description, xacro)
@@ -7,13 +7,12 @@
 <xacro:include filename="$(find reppy_bot_urdf)/urdf/diff_drive_setup.xacro"/>
 <!-- Simple Robot Settings -->
-	<xacro:property name="wheel_diameter" value="0.05"/>
-	<xacro:property name="wheel_width" value="0.01"/>
-	<xacro:property name="wheel_base_center_x" value="-0.02"/>
-	<xacro:property name="wheel_separation" value="0.10"/>
-	<xacro:property name="chassis_width"  value="0.07"/>
-	<xacro:property name="chassis_len"    value="0.09"/>
-	<xacro:property name="chassis_height" value="0.04"/>
-    <xacro:property name="chassis_floor_clearance" value="0.02"/>
-    <xacro:property name="caster_collision_x" value="0.02"/>
+<xacro:property name="chassis_height" value="0.15"/>
+<xacro:property name="chassis_width"  value="${chassis_height*1.618}"/>
+<xacro:property name="chassis_len"    value="${chassis_width+chassis_height}"/>
+<xacro:property name="chassis_floor_clearance" value="${chassis_height/(1.618*2)}"/>
+<xacro:property name="wheel_diameter" value="${chassis_len/(1.618*1.618)}"/>
+<xacro:property name="wheel_width" value="${chassis_width/(16.18)}"/>
+<xacro:property name="wheel_base_center_x" value="${chassis_len/(-1.618*3)}"/>
+<xacro:property name="caster_collision_x" value="${chassis_len/(1.618*2)}"/>
 <link name="base_link"/>
 <link name="chassis">
@@ -22,4 +21,7 @@
 			<box size="${chassis_len} ${chassis_width} ${chassis_height}" />
 		</geometry>
+		<material name="Green">
+			<color rgba="0 1 0 1"/>
+		</material>
 	</visual>
 	<collision>
@@ -28,10 +30,17 @@
 		</geometry>
 	</collision>
-	<material>
-		<color rgba="0.0 0.0 1.0 1.0"/>
-	</material>
+	<inertial>
+            <mass value="1.0"/>
+            <origin xyz="0.0 0.0 0.0"/>
+            <inertia ixx="0.1"
+                     iyy="0.1"
+                     izz="0.1"
+  	            	 iyz="0.0"
+		             ixy="0.0"
+		             ixz="0.0"/>
+    </inertial>
 </link>
 <gazebo reference="chassis">
-	<material name="Gazebo/Blue"/>
+	<material value="Gazebo/Green"/>
 </gazebo>
 <joint name="base_chassis_joint" type="fixed">
@@ -45,4 +54,7 @@
 			<sphere radius="${chassis_floor_clearance}" />
 		</geometry>
+		<material name="Black">
+			<color rgba="0 0 0 1"/>
+		</material>
 	</visual>
 	<collision>
@@ -51,10 +63,17 @@
 		</geometry>
 	</collision>
-	<material>
-		<color rgba="0.0 0.0 1.0 1.0"/>
-	</material>
+    <inertial>
+    <mass value="1.0"/>
+    <origin xyz="0.0 0.0 0.0"/>
+    <inertia ixx="0.1"
+             iyy="0.1"
+             izz="0.1"
+        	 iyz="0.0"
+             ixy="0.0"
+             ixz="0.0"/>
+    </inertial>
 </link>
 <gazebo reference="caster_collision">
-	<material name="Gazebo/FlatBlack"/>
+	<material value="Gazebo/FlatBlack"/>
 </gazebo>
 <joint name="base_caster_col_joint" type="fixed">
@@ -66,5 +85,5 @@
 	 base_frame="base_link"
 	 robot_namespace=""
-	 wheel_base_center_x="-0.02"
+	 wheel_base_center_x="${wheel_base_center_x}"
      wheel_separation ="${chassis_width}"
      wheel_diameter="${wheel_diameter}"
@@ -76,6 +95,6 @@
 	 wheel_friction1="100000"
      wheel_friction2="1000"
-	 wheel_contact_damping="10"
-     wheel_contact_stiffness="10"
+	 wheel_contact_damping="100.0"
+     wheel_contact_stiffness="1000000.0"
 	 wheel_mass="3"
      cmd_topic="/cmd_vel"

Commit message: bumper tests

File: reppy_bot_urdf/urdf/test_bot.xacro (robot description, xacro)
@@ -54,4 +54,31 @@
 	<origin xyz="0 0 ${chassis_floor_clearance+chassis_height/2}" rpy="0 0 0" />
 </joint>
+<!--
+ <link name="bumper0">
+	<visual>
+		<geometry>
+			<box size="0.1 0.1 0.1" />
+		</geometry>
+	</visual>
+	<collision name="bump_col">
+		<geometry>
+			<box size="0.1 0.1 0.1" />
+		</geometry>
+	</collision>
+</link>
+<joint name="chassis_bumper_joint" type="fixed">
+	<parent link="chassis" />
+	<child link="bumper0" />
+	<origin xyz="1 0 0" rpy="0 0 0" />
+</joint>
+<gazebo reference="bumper0">
+  <plugin name="bumper0_controller" filename="libgazebo_ros_bumper.so">
+    <alwaysOn>true</alwaysOn>
+    <updateRate>30</updateRate>
+    <bumperTopicName>/bumper0</bumperTopicName>
+    <frameName>world</frameName>
+  </plugin>
+</gazebo>
+-->
 <link name="caster_collision">
 	<visual>

Commit message: add macros to bot

File: reppy_bot_urdf/urdf/test_bot.xacro (robot description, xacro)
@@ -21,4 +21,5 @@
 <xacro:property name="robot_namespace" value="/" />
 <link name="base_link" />
+<!--CHASSIS-->
 <link name="chassis">
 	<visual>
@@ -54,31 +55,5 @@
 	<origin xyz="0 0 ${chassis_floor_clearance+chassis_height/2}" rpy="0 0 0" />
 </joint>
-<!--
- <link name="bumper0">
-	<visual>
-		<geometry>
-			<box size="0.1 0.1 0.1" />
-		</geometry>
-	</visual>
-	<collision name="bump_col">
-		<geometry>
-			<box size="0.1 0.1 0.1" />
-		</geometry>
-	</collision>
-</link>
-<joint name="chassis_bumper_joint" type="fixed">
-	<parent link="chassis" />
-	<child link="bumper0" />
-	<origin xyz="1 0 0" rpy="0 0 0" />
-</joint>
-<gazebo reference="bumper0">
-  <plugin name="bumper0_controller" filename="libgazebo_ros_bumper.so">
-    <alwaysOn>true</alwaysOn>
-    <updateRate>30</updateRate>
-    <bumperTopicName>/bumper0</bumperTopicName>
-    <frameName>world</frameName>
-  </plugin>
-</gazebo>
--->
+<!--CASTER -->
 <link name="caster_collision">
 	<visual>
@@ -140,4 +115,36 @@
 	 ros_plugin_publish_wheel_tf="true"
 	 ros_plugin_publish_tf="1" />
+<!-- BUMPER -->
+<link name="bumper0">
+	<visual>
+		<geometry>
+			<box size="0.1 0.1 0.1" />
+		</geometry>
+	</visual>
+	<collision name="bumper0_collision">
+		<geometry>
+			<box size="0.1 0.1 0.1" />
+		</geometry>
+	</collision>
+</link>
+<joint name="chassis_bumper_joint" type="fixed">
+	<parent link="chassis" />
+	<child link="bumper0" />
+	<origin xyz="${chassis_len/2}  ${chassis_width/2} 0" rpy="0 0 0" />
+	<axis xyz="0 1 0"/>
+</joint>
+<gazebo reference="bumper0">
+  <sensor name="bumper0_sensor" type="contact">
+    <always_on>true</always_on>
+    <update_rate>30</update_rate>
+    <contact>
+      <collision>bumper0_collision</collision>
+    </contact>
+    <plugin name="bumper0_plugin" filename="libgazebo_ros_bumper.so">
+      <bumperTopicName>bumper0_sensor_state</bumperTopicName>
+      <frameName>bumper0</frameName>
+    </plugin>
+  </sensor>
+</gazebo>
 <xacro:gps_receiver
 		id="0"
@@ -164,4 +171,10 @@
 		yaw="0"
 		gaussian_noise="2.89e-08"
+		imu_x="0"
+		imu_y="0"
+		imu_z="0"
+		imu_roll="0"
+		imu_pitch="0"
+		imu_yaw="0"
 		/>
 <xacro:rplidar id="0"

Commit message: bumper ready to use

File: reppy_bot_urdf/urdf/test_bot.xacro (robot description, xacro)
@@ -11,4 +11,5 @@
 <xacro:include filename="$(find reppy_bot_urdf)/urdf/rplidar.xacro"			/>
 <xacro:include filename="$(find reppy_bot_urdf)/urdf/camera.xacro"			/>
+<xacro:include filename="$(find reppy_bot_urdf)/urdf/bumper.xacro"			/>
 <!-- Simple Robot Settings -->
 <xacro:property name="chassis_height"          value="0.15"                            />
@@ -21,7 +22,9 @@
 <xacro:property name="caster_collision_x"      value="${chassis_len/(1.618*2)}"        />
 <xacro:property name="robot_namespace" value="/" />
-<link name="base_link" />
 <!--CHASSIS-->
 <link name="chassis">
+	 <xacro:inertia_box x="${chassis_len}" y="${chassis_width}" z="${chassis_height}" mass="1">
+      <origin xyz="0 0 0" rpy="0 0 0" />
+    </xacro:inertia_box>
 	<visual>
 		<geometry>
@@ -37,24 +40,24 @@
 		</geometry>
 	</collision>
-	<inertial>
-            <mass value="1.0"/>
-            <origin xyz="0.0 0.0 0.0"/>
-            <inertia ixx="0.1"
-                     iyy="0.1"
-                     izz="0.1"
-  	            	 iyz="0.0"
-		             ixy="0.0"
-		             ixz="0.0"/>
-    </inertial>
 </link>
 <gazebo reference="chassis">
 	<material value="Gazebo/Green"/>
 </gazebo>
-<joint name="base_chassis_joint" type="fixed">
-	<parent link="base_link" />
-	<child link="chassis" />
-	<origin xyz="0 0 ${chassis_floor_clearance+chassis_height/2}" rpy="0 0 0" />
-</joint>
-<!--CASTER -->
+<xacro:bumper name="bumper0" parent="chassis" always_on="true" update_rate="30" topic="bumper0"  has_inertia="true">
+	<origin xyz="${chassis_len/2} ${chassis_width/2} 0" rpy="0 0 0" />
+	<geometry>
+		<box size="0.1 0.1 0.1" />
+	</geometry>
+	<material name="Green">
+		<color rgba="0 1 0 0.5"/>
+	</material>
+	 <xacro:inertia_box x="0.1" y="0.1" z="0.1" mass="0.1">
+      <origin xyz="0 0 0" rpy="0 0 0" />
+    </xacro:inertia_box>
+</xacro:bumper>
+<gazebo reference="bumper0">
+	<material value="Gazebo/FlatBlack" />
+</gazebo>
+<!--CASTER
 <link name="caster_collision">
 	<visual>
@@ -82,4 +85,6 @@
     </inertial>
 </link>
+-->
+<!--
 <gazebo reference="caster_collision">
 	<material value="Gazebo/FlatBlack"/>
@@ -116,36 +121,6 @@
 	 ros_plugin_publish_wheel_tf="true"
 	 ros_plugin_publish_tf="1" />
-<!-- BUMPER -->
-<link name="bumper0">
-	<visual>
-		<geometry>
-			<box size="0.1 0.1 0.1" />
-		</geometry>
-	</visual>
-	<collision name="bumper0_collision">
-		<geometry>
-			<box size="0.1 0.1 0.1" />
-		</geometry>
-	</collision>
-</link>
-<joint name="chassis_bumper_joint" type="fixed">
-	<parent link="chassis" />
-	<child link="bumper0" />
-	<origin xyz="${chassis_len/2}  ${chassis_width/2} 0" rpy="0 0 0" />
-	<axis xyz="0 1 0"/>
-</joint>
-<gazebo reference="bumper0">
-  <sensor name="bumper0_sensor" type="contact">
-    <always_on>true</always_on>
-    <update_rate>30</update_rate>
-    <contact>
-      <collision>bumper0_collision</collision>
-    </contact>
-    <plugin name="bumper0_plugin" filename="libgazebo_ros_bumper.so">
-      <bumperTopicName>bumper0_sensor_state</bumperTopicName>
-      <frameName>bumper0</frameName>
-    </plugin>
-  </sensor>
-</gazebo>
+	-->
+	 	<!--
 <xacro:gps_receiver
 		id="0"
@@ -221,3 +196,4 @@
 		update_rate      ="30"
         />
+        	-->
 </robot>

Commit message: add bumpers

File: reppy_bot_urdf/urdf/test_bot.xacro (robot description, xacro)
@@ -13,5 +13,5 @@
 <xacro:include filename="$(find reppy_bot_urdf)/urdf/bumper.xacro"			/>
 <!-- Simple Robot Settings -->
-<xacro:property name="chassis_height"          value="0.15"                            />
+<xacro:property name="chassis_height"          value="0.25"                            />
 <xacro:property name="chassis_width"           value="${chassis_height*1.618}"         />
 <xacro:property name="chassis_len"             value="${chassis_width+chassis_height}" />
@@ -25,5 +25,5 @@
 <link name="chassis">
 	 <xacro:inertia_box x="${chassis_len}" y="${chassis_width}" z="${chassis_height}" mass="1">
-      <origin xyz="0 0 0" rpy="0 0 0" />
+      <origin xyz="0 0 ${chassis_floor_clearance}" rpy="0 0 0" />
     </xacro:inertia_box>
 	<visual>
@@ -47,14 +47,44 @@
 	<origin xyz="${chassis_len/2} ${chassis_width/2} 0" rpy="0 0 0" />
 	<geometry>
-		<box size="0.1 0.1 0.1" />
+		<box size="0.02 0.02 ${chassis_height}" />
 	</geometry>
-	<material name="Green">
-		<color rgba="0 1 0 0.5"/>
+	<material name="Black">
+		<color rgba="0 0 0 1"/>
 	</material>
-	 <xacro:inertia_box x="0.1" y="0.1" z="0.1" mass="0.1">
+	 <xacro:inertia_box x="0.02" y="0.02" z="${chassis_height}" mass="0.1">
       <origin xyz="0 0 0" rpy="0 0 0" />
     </xacro:inertia_box>
 </xacro:bumper>
 <gazebo reference="bumper0">
+	<material value="Gazebo/FlatBlack" />
+</gazebo>
+<xacro:bumper name="bumper1" parent="chassis" always_on="true" update_rate="30" topic="bumper0"  has_inertia="true">
+	<origin xyz="${chassis_len/2} -${chassis_width/2} 0" rpy="0 0 0" />
+	<geometry>
+		<box size="0.02 0.02 ${chassis_height}" />
+	</geometry>
+	<material name="Black">
+		<color rgba="0 0 0 1"/>
+	</material>
+	 <xacro:inertia_box x="0.02" y="0.02" z="${chassis_height}" mass="0.1">
+      <origin xyz="0 0 0" rpy="0 0 0" />
+    </xacro:inertia_box>
+</xacro:bumper>
+<gazebo reference="bumper1">
+	<material value="Gazebo/FlatBlack" />
+</gazebo>
+<xacro:bumper name="bumper2" parent="chassis" always_on="true" update_rate="30" topic="bumper0"  has_inertia="true">
+	<origin xyz="${chassis_len/2} 0 -${chassis_height/4}" rpy="0 0 0" />
+	<geometry>
+		<box size="0.02 ${chassis_width-0.04} 0.02" />
+	</geometry>
+	<material name="Black">
+		<color rgba="0 0 0 1"/>
+	</material>
+	 <xacro:inertia_box x="0.02" y="0.02" z="0.04" mass="0.1">
+      <origin xyz="0 0 0" rpy="0 0 0" />
+    </xacro:inertia_box>
+</xacro:bumper>
+<gazebo reference="bumper2">
 	<material value="Gazebo/FlatBlack" />
 </gazebo>
